File: hardware/front-array/front-array.kicad_pcb (KiCad board)
At the start: 2 copper layers, 96 x 22 mm, 6 parts, among them J1 Conn_01x05, J2 Conn_01x05, U1 VL53L0X, U2 VL53L0X

Commit message: 3d modeling update
Other:
- board text added: "JLCJLCJLCJLC"
Changed lines of the file:
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@@
-(kicad_pcb (version 20210424) (generator pcbnew)
+(kicad_pcb (version 20210722) (generator pcbnew)
   (general
     (thickness 1.6)
@@
     (property "Sheetname" "")
     (attr through_hole)
-    (fp_text reference "J1" (at -4.38 -2.77 90) (layer "F.SilkS")
+    (fp_text reference "J1" (at -4.380005 -2.769992 90) (layer "F.SilkS") hide
       (effects (font (size 1 1) (thickness 0.15)))
     )
@@
     (property "Sheetname" "")
     (attr through_hole)
-    (fp_text reference "J2" (at -4.38 -2.77 90) (layer "F.SilkS")
+    (fp_text reference "J2" (at -4.380005 -2.769992 90) (layer "F.SilkS") hide
       (effects (font (size 1 1) (thickness 0.15)))
     )
@@
   (gr_line (start 117 86) (end 102 86) (layer "Edge.Cuts") (width 0.1))
   (gr_line (start 117 100) (end 183 100) (layer "Edge.Cuts") (width 0.1))
+  (gr_text "JLCJLCJLCJLC" (at 150.254 98.476) (layer "B.SilkS")
+    (effects (font (size 1 1) (thickness 0.15)) (justify mirror))
+  )
   (segment (start 104.534 80.442) (end 104.534 81.458) (width 0.25) (layer "F.Cu") (net 1))
   (segment (start 105.22 81.8) (end 105.22 82.906) (width 0.25) (layer "F.Cu") (net 1))
