File: hardware/mainboard/mainboard.kicad_sch (KiCad schematic)
At the start: 66 parts, among them J1 Conn_01x14, J10 Conn_01x14, J11 Conn_01x14, J12 Conn_02x06_Odd_Even, J13 Conn_01x14, J14 Conn_01x14, J15 Conn_01x14, J16 Conn_01x01, J17 Conn_01x01, J18 Conn_01x03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

Commit message: docs update
Parts:
- R1: value 1K -> 2.2K
