File: hardware/top_plate/top_plate.kicad_sch (KiCad schematic)
At the start: 17 parts, among them J1 Conn_01x04_Male, J2 Conn_01x04, J3 Conn_02x04_Odd_Even, J4 Conn_01x04, Q1 BSS138, Q2 BSS138, SW1 SW_Push, SW2 SW_Push, U1 AP2112K-1.8, U2 ICM-20948

Commit message: Creating v4 branch
Parts:
- removed C1, C2: 1uF, Capacitor_SMD:C_0805_2012Metric, symbol Device:C
- removed C3, C4, C5: 100nF, Capacitor_SMD:C_0603_1608Metric, symbol Device:C
- removed J1: Conn_01x04_Male, shurik-personal:OLED_128x64_1_3in, symbol Connector:Conn_01x04_Male
- removed J2, J4: Conn_01x04, Connector_JST:JST_SH_SM04B-SRSS-TB_1x04-1MP_P1.00mm_Horizontal, symbol Connector_Generic:Conn_01x04
- removed J3: Conn_02x04_Odd_Even, Connector_PinSocket_2.54mm:PinSocket_2x04_P2.54mm_Vertical, symbol Connector_Generic:Conn_02x04_Odd_Even
- removed Q1, Q2: BSS138, Package_TO_SOT_SMD:SOT-23, symbol Transistor_FET:BSS138
- removed R1, R2: 10K, Resistor_SMD:R_0603_1608Metric, symbol Device:R
- removed SW1, SW2: SW_Push, Button_Switch_THT:SW_PUSH_6mm_H4.3mm, symbol Switch:SW_Push
- removed U1: AP2112K-1.8, Package_TO_SOT_SMD:SOT-23-5, symbol Regulator_Linear:AP2112K-1.8
- removed U2: ICM-20948, Sensor_Motion:InvenSense_QFN-24_3x3mm_P0.4mm, symbol Sensor_Motion:ICM-20948
- added A1: Adafruit_Feather_Generic, Module:Adafruit_Feather, symbol MCU_Module:Adafruit_Feather_Generic
- added BZ1: Buzzer, Buzzer_Beeper:Buzzer_TDK_PS1240P02BT_D12.2mm_H6.5mm, symbol Device:Buzzer
- added C1, C2: 100nF, Capacitor_SMD:C_0603_1608Metric, symbol Device:C_Small
- added D1, D2: SK6812MINI, LED_SMD:LED_SK6812MINI_PLCC4_3.5x3.5mm_P1.75mm, symbol LED:SK6812MINI
- added J1, J3: Conn_01x05, Connector_PinHeader_2.54mm:PinHeader_1x05_P2.54mm_Horizontal, symbol Connector_Generic:Conn_01x05
- added J10: Conn_02x04_Odd_Even, Connector_PinHeader_2.54mm:PinHeader_2x04_P2.54mm_Vertical, symbol Connector_Generic:Conn_02x04_Odd_Even
- added J2: Conn_02x06_Odd_Even, Connector_PinSocket_2.54mm:PinSocket_2x06_P2.54mm_Vertical, symbol Connector_Generic:Conn_02x06_Odd_Even
- added J5: Conn_01x04, Connector_JST:JST_PH_B4B-PH-K_1x04_P2.00mm_Vertical, symbol Connector_Generic:Conn_01x04
- added J6, J7: Conn_01x04, shurik-personal:connector-4p-generic-nosilk, symbol Connector_Generic:Conn_01x04
- added J8, J9: Conn_01x04, Connector_JST:JST_SH_BM04B-SRSS-TB_1x04-1MP_P1.00mm_Vertical, symbol Connector_Generic:Conn_01x04
- added R1, R2: 3.3K, Resistor_SMD:R_0603_1608Metric, symbol Device:R_Small
Connections:
- net +3V3: now also J10.3 (Pin_3), J10.4 (Pin_4), J2.12 (Pin_12), J3.5 (Pin_5), J6.1 (Pin_1), J8.2 (Pin_2), J9.2 (Pin_2), R1.1, R2.1
- net SCL: now also A1.18 (SCL), J2.9 (Pin_9), J3.3 (Pin_3), J5.2 (Pin_2), J7.2 (Pin_2), J8.4 (Pin_4), J9.4 (Pin_4), R1.2
- net SDA: now also A1.17 (SDA), J2.11 (Pin_11), J3.4 (Pin_4), J5.1 (Pin_1), J7.1 (Pin_1), J8.3 (Pin_3), J9.3 (Pin_3), R2.2
- new net: D1.1 (DOUT), D2.3 (DIN)
- new net A1: A1.6 (A1), J10.6 (Pin_6)
- new net A2: A1.7 (A2), J10.8 (Pin_8)
- new net A3: A1.8 (A3), J2.4 (Pin_4)
- new net A4: A1.9 (A4), J2.5 (Pin_5)
- new net A5: A1.10 (A5), J2.6 (Pin_6)
- new net D10: A1.22 (D3), J6.2 (Pin_2)
- new net D11-XSHUT2: A1.23 (D4), J1.2 (Pin_2)
- new net D12: A1.24 (D5), J1.3 (Pin_3)
- new net D13-BUZZ: A1.25 (D6), BZ1.1 (-)
- new net D5-XSHUT1: A1.19 (D0), J3.2 (Pin_2)
- new net D6: A1.20 (D1)
- new net D9: A1.21 (D2), J6.3 (Pin_3)
- new net GND: A1.4 (GND), BZ1.2 (+), C1.2, C2.2, D1.2 (VSS), D2.2 (VSS), J1.1 (Pin_1), J10.1 (Pin_1), J10.2 (Pin_2), J2.1 (Pin_1), J3.1 (Pin_1), J5.3 (Pin_3), J6.4 (Pin_4), J7.3 (Pin_3), J8.1 (Pin_1), J9.1 (Pin_1)
- new net MISO: A1.13 (MISO), J2.10 (Pin_10)
- new net MOSI: A1.12 (MOSI), J2.8 (Pin_8)
- new net NEOPXL: A1.5 (A0), D1.3 (DIN)
- new net RESET: A1.1 (~{RESET}), J2.3 (Pin_3)
- new net RX: A1.14 (RX), J10.7 (Pin_7)
- new net SCK: A1.11 (SCK), J2.7 (Pin_7)
- new net TX: A1.15 (TX), J10.5 (Pin_5)
- new net VCC: A1.28 (VBAT), C1.1, C2.1, D1.4 (VDD), D2.4 (VDD), J1.5 (Pin_5), J2.2 (Pin_2), J5.4 (Pin_4), J7.4 (Pin_4)
- new net VUSB: A1.26 (USB)
Other:
- note added: "Adafruit ESP32-S3 Feather"
- note added: "Analog connectors"
- note added: "Buzzer"
- note added: "Connector to main board"
- note added: "Distance sensors connector"
- note added: "Huskylens connector"
- note added: "NeoPixels"
- note added: "Qwiic I2C connectors"
- note added: "Sonar connector"
- company: (none) -> Island Robotics
- title: (none) -> Yozh top plate

Commit message: Updating license information
Other:
- company: Island Robotics -> Alexander Kirillov
Changed lines of the file:
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@@
   (title_block
     (title "Yozh top plate")
-    (date "2023-10-26")
+    (date "2023-10-28")
     (rev "4.02")
-    (company "Island Robotics")
+    (company "Alexander Kirillov")
+    (comment 1 "shurik179@gmail.com")
   )
   (junction (at 172.72 93.98) (diameter 0) (color 0 0 0 0)
