File: hardware/distance_sensors/distance_sensors.kicad_sch (KiCad schematic)
At the start: 12 parts, among them J1 Conn_01x05, J2 Conn_01x05, U1 VL53L0X, U2 VL53L0X

Commit message: Updating license information
Other:
- company: Island Robotics -> Alexander Kirillov
Changed lines of the file:
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@@
   (title_block
     (title "Distance sensor board")
-    (date "2023-10-26")
+    (date "2023-10-28")
     (rev "4.02")
-    (company "Island Robotics")
+    (company "Alexander Kirillov")
+    (comment 1 "shurik179@gmail.com")
   )
   (junction (at 34.29 137.16) (diameter 0) (color 0 0 0 0)
