File: hardware/mainboard_dual_battery/boost.kicad_sch (KiCad schematic)
At the start: 14 parts, among them U14 PAM2423

Commit message: Updating license information
Other:
- company: Island Robotics -> Alexander Kirillov
Changed lines of the file:
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@@
   (title_block
     (title "Yozh mainboard")
-    (date "2023-10-26")
+    (date "2023-10-28")
     (rev "4.02")
-    (company "Island Robotics")
+    (company "Alexander Kirillov")
+    (comment 1 "shurik179@gmail.com")
   )
   (junction (at 161.29 74.93) (diameter 0) (color 0 0 0 0)
