File: hardware/mainboard_dual_battery/mainboard_dual_battery.kicad_sch (KiCad schematic)
At the start: 53 parts, among them J1 Conn_01x05, J10 Conn_01x05, J11 Conn_01x03, J12 Conn_01x03, J13 Conn_02x06_Odd_Even, J14 Conn_01x02, J2 Conn_01x05, J3 USB_B_Micro, J4 Conn_01x01, J5 Conn_01x01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

Commit message: Updating license information
Other:
- company: Island Robotics -> Alexander Kirillov
Changed lines of the file:
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@@
   (title_block
     (title "Yozh mainboard")
-    (date "2023-10-26")
+    (date "2023-10-28")
     (rev "4.02")
-    (company "Island Robotics")
+    (company "Alexander Kirillov")
+    (comment 1 "shurik179@gmail.com")
   )
   (junction (at 234.95 85.09) (diameter 0.9144) (color 0 0 0 0)
