File: hardware/mainboard_dual_battery/reflectance_array.kicad_sch (KiCad schematic)
At the start: 19 parts, among them U10 AP3019A, U2 ITR9909, U3 ITR9909, U4 ITR9909, U5 ITR9909, U6 ITR9909, U7 ITR9909, U8 ITR9909

Commit message: Updating license information
Other:
- company: Island Robotics -> Alexander Kirillov
Changed lines of the file:
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@@
   (title_block
     (title "Yozh mainboard")
-    (date "2023-10-26")
+    (date "2023-10-28")
     (rev "4.02")
-    (company "Island Robotics")
+    (company "Alexander Kirillov")
+    (comment 1 "shurik179@gmail.com")
   )
   (junction (at 73.66 63.5) (diameter 0.9144) (color 0 0 0 0)
